File: kicad_pcb.kicad_pcb (KiCad board)
At the start: 2 copper layers, 285 x 95.1 mm, 123 parts, among them J1 USB_B_Mini, SW1 SW_Push, U1 ATmega32U4-AU, Y1 16Mhz

Commit message: Ordered all keyboard rows
Parts:
- added MX31: MX-1U, MX_Alps_Hybrid:MXOnly-1U-NoLED, F.Cu at (77.8, 87.3)
- added MX32: MX-1U, MX_Alps_Hybrid:MXOnly-1U-NoLED, F.Cu at (96.8, 87.3)
- added MX33: MX-1U, MX_Alps_Hybrid:MXOnly-1U-NoLED, F.Cu at (115.9, 87.3)
- added MX34: MX-1U, MX_Alps_Hybrid:MXOnly-1U-NoLED, F.Cu at (134.9, 87.3)
- added MX35: MX-1U, MX_Alps_Hybrid:MXOnly-1U-NoLED, F.Cu at (154.0, 87.3)
- added MX36: MX-1U, MX_Alps_Hybrid:MXOnly-1U-NoLED, F.Cu at (173.0, 87.3)
- added MX37: MX-1U, MX_Alps_Hybrid:MXOnly-1U-NoLED, F.Cu at (192.1, 87.3)
- added MX38: MX-1U, MX_Alps_Hybrid:MXOnly-1U-NoLED, F.Cu at (219.1, 6.35)
- added MX39: MX-1U, MX_Alps_Hybrid:MXOnly-1U-NoLED, F.Cu at (220.7, 87.3)
- added MX40: MX-1U, MX_Alps_Hybrid:MXOnly-1U-NoLED, F.Cu at (239.7, 87.3)
- added MX41: MX-1U, MX_Alps_Hybrid:MXOnly-1U-NoLED, F.Cu at (258.8, 87.3)
- added MX42: MX-1U, MX_Alps_Hybrid:MXOnly-1U-NoLED, F.Cu at (277.8, 87.3)
- added MX43: MX-1U, MX_Alps_Hybrid:MXOnly-1U-NoLED, F.Cu at (296.9, 87.3)
- added MX44: MX-1U, MX_Alps_Hybrid:MXOnly-1U-NoLED, F.Cu at (315.9, 87.3)
- added MX45: MX-1U, MX_Alps_Hybrid:MXOnly-1U-NoLED, F.Cu at (335.0, 87.3)
- added MX46: MX-1U, MX_Alps_Hybrid:MXOnly-1U-NoLED, F.Cu at (73.0, 106.4)
- added MX47: MX-1U, MX_Alps_Hybrid:MXOnly-1U-NoLED, F.Cu at (92.1, 106.4)
- added MX48: MX-1U, MX_Alps_Hybrid:MXOnly-1U-NoLED, F.Cu at (111.1, 106.4)
- added MX49: MX-1U, MX_Alps_Hybrid:MXOnly-1U-NoLED, F.Cu at (130.2, 106.4)
- added MX50: MX-1U, MX_Alps_Hybrid:MXOnly-1U-NoLED, F.Cu at (149.2, 106.4)
- added MX51: MX-1U, MX_Alps_Hybrid:MXOnly-1U-NoLED, F.Cu at (168.3, 106.4)
- added MX52: MX-1U, MX_Alps_Hybrid:MXOnly-1U-NoLED, F.Cu at (187.3, 106.4)
- added MX53: MX-1U, MX_Alps_Hybrid:MXOnly-1U-NoLED, F.Cu at (206.4, 106.4)
- added MX54: MX-1U, MX_Alps_Hybrid:MXOnly-1U-NoLED, F.Cu at (225.4, 106.4)
- added MX55: MX-1U, MX_Alps_Hybrid:MXOnly-1U-NoLED, F.Cu at (244.5, 106.4)
- added MX56: MX-1U, MX_Alps_Hybrid:MXOnly-1U-NoLED, F.Cu at (263.5, 106.4)
- added MX57: MX-1U, MX_Alps_Hybrid:MXOnly-1U-NoLED, F.Cu at (282.6, 106.4)
- added MX58: MX-1U, MX_Alps_Hybrid:MXOnly-1U-NoLED, F.Cu at (301.6, 106.4)
- added MX59: MX-1U, MX_Alps_Hybrid:MXOnly-1U-NoLED, F.Cu at (320.7, 106.4)
- added MX60: MX-1U, MX_Alps_Hybrid:MXOnly-1U-NoLED, F.Cu at (339.7, 106.4)
- added MX61: MX-1U, MX_Alps_Hybrid:MXOnly-1U-NoLED, F.Cu at (73.0, 125.4)
- added MX62: MX-1U, MX_Alps_Hybrid:MXOnly-1U-NoLED, F.Cu at (92.1, 125.4)
- added MX63: MX-1U, MX_Alps_Hybrid:MXOnly-1U-NoLED, F.Cu at (111.1, 125.4)
- added MX64: MX-1U, MX_Alps_Hybrid:MXOnly-1U-NoLED, F.Cu at (130.2, 125.4)
- added MX65: MX-1U, MX_Alps_Hybrid:MXOnly-1U-NoLED, F.Cu at (149.2, 125.4)
- added MX66: MX-1U, MX_Alps_Hybrid:MXOnly-1U-NoLED, F.Cu at (168.3, 125.4)
- added MX67: MX-1U, MX_Alps_Hybrid:MXOnly-1U-NoLED, F.Cu at (187.3, 125.4)
- added MX68: MX-1U, MX_Alps_Hybrid:MXOnly-1U-NoLED, F.Cu at (206.4, 125.4)
- added MX69: MX-1U, MX_Alps_Hybrid:MXOnly-1U-NoLED, F.Cu at (225.4, 125.4)
- added MX70: MX-1U, MX_Alps_Hybrid:MXOnly-1U-NoLED, F.Cu at (244.5, 125.4)
- added MX71: MX-1U, MX_Alps_Hybrid:MXOnly-1U-NoLED, F.Cu at (263.5, 125.4)
- added MX72: MX-1U, MX_Alps_Hybrid:MXOnly-1U-NoLED, F.Cu at (282.6, 125.4)
- added MX73: MX-1U, MX_Alps_Hybrid:MXOnly-1U-NoLED, F.Cu at (301.6, 125.4)
- added MX74: MX-1U, MX_Alps_Hybrid:MXOnly-1U-NoLED, F.Cu at (320.7, 125.4)
- added MX75: MX-1U, MX_Alps_Hybrid:MXOnly-1U-NoLED, F.Cu at (339.7, 125.4)
- moved MX23 41.3 mm to (206.4, 27.0)
- moved MX29 9.53 mm to (311.1, 68.3), turned to 0 degrees
- moved MX30 9.53 mm to (330.2, 68.3)
- moved MX18 9.53 mm to (120.7, 68.3)
- moved MX20 9.53 mm to (158.8, 68.3)
- moved MX21 9.53 mm to (177.8, 68.3)
- moved MX22 9.53 mm to (196.8, 68.3)
- moved MX24 9.53 mm to (215.9, 68.3)
- moved MX25 9.53 mm to (234.9, 68.3)
- moved MX16 9.52 mm to (82.5, 68.3)
- moved MX17 9.52 mm to (101.6, 68.3), turned to 0 degrees
- moved MX19 9.52 mm to (139.7, 68.3)
- moved MX26 9.52 mm to (254.0, 68.3)
- moved MX27 9.52 mm to (273.1, 68.3)
- moved MX28 9.52 mm to (292.1, 68.3)

Commit message: placed all the diodes
Parts:
- MX17: value TAB -> Q
- MX18: value Q -> W
- MX19: value W -> E
- MX20: value E -> R
- MX21: value R -> T
- MX22: value T -> [
- MX24: value U -> ]
- MX25: value I -> Y
- MX26: value O -> U
- MX27: value P -> I
- MX28: value [ -> O
- MX29: value ] -> P
- MX31: value MX-1U -> LAYER_UP
- MX32: value MX-1U -> A
- MX33: value MX-1U -> S
- MX34: value MX-1U -> D
- MX35: value MX-1U -> F
- MX36: value MX-1U -> G
- MX37: value MX-1U -> HOME
- MX39: value MX-1U -> PAGE UP
- MX40: value MX-1U -> H
- MX41: value MX-1U -> J
- MX42: value MX-1U -> K
- MX43: value MX-1U -> L
- MX44: value MX-1U -> SEMI COLON
- MX45: value MX-1U -> RETURN
- MX46: value MX-1U -> L SHIFT
- MX47: value MX-1U -> Z
- MX48: value MX-1U -> X
- MX49: value MX-1U -> C
- MX50: value MX-1U -> V
- MX51: value MX-1U -> B
- MX52: value MX-1U -> END
- MX53: value MX-1U -> DELETE
- MX54: value MX-1U -> PAGE DOWN
- MX55: value MX-1U -> N
- MX56: value MX-1U -> M
- MX57: value MX-1U -> COMMA
- MX58: value MX-1U -> FULL STOP
- MX62, MX63, MX64: footprint MX_Alps_Hybrid:MXOnly-1U-NoLED -> MX_Alps_Hybrid:MXOnly-1.25U-NoLED
- MX65: footprint MX_Alps_Hybrid:MXOnly-1U-NoLED -> MX_Alps_Hybrid:MXOnly-2.25U-NoLED
- MX70: footprint MX_Alps_Hybrid:MXOnly-1U-NoLED -> MX_Alps_Hybrid:MXOnly-2U-NoLED
- moved D69 243.4 mm to (-1.59, 31.1), turned to 90 degrees
- moved D66 235.3 mm to (-11.1, 54.1), turned to 90 degrees
- moved D38 227.6 mm to (22.2, 54.9), turned to 90 degrees
- moved D67 218.9 mm to (11.1, 45.4), turned to 90 degrees
- moved D46 206.5 mm to (66.7, 113.7), turned to 90 degrees
- moved D47 199.4 mm to (85.7, 113.7), turned to 90 degrees
- moved D75 198.3 mm to (346.1, 131.1), turned to 90 degrees
- moved MX69 194.2 mm to (137.3, -47.6)
- moved D48 191.4 mm to (104.8, 113.7), turned to 90 degrees
- moved D74 190.0 mm to (327.0, 131.1), turned to 90 degrees
- moved D16 189.8 mm to (76.2, 75.5), turned to 90 degrees
- moved MX66 186.3 mm to (99.2, -47.6)
- moved MX67 186.3 mm to (118.3, -47.6)
- moved D49 184.4 mm to (123.8, 113.7), turned to 90 degrees
- moved D61 182.3 mm to (66.7, 131.8), turned to 90 degrees
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Connections:
- D46 pad 1: ROW3 -> COL5
- D47 pad 1: ROW3 -> COL5
- D48 pad 1: ROW3 -> COL5
- D49 pad 1: ROW3 -> COL5
- D50 pad 1: ROW3 -> COL5
- D51 pad 1: ROW3 -> COL5
- D52 pad 1: ROW3 -> COL5
- D53 pad 1: ROW3 -> COL5
- D54 pad 1: ROW3 -> COL5
- D55 pad 1: ROW3 -> COL5
- D56 pad 1: ROW3 -> COL5
- D57 pad 1: ROW3 -> COL5
- D58 pad 1: ROW3 -> COL5
- D59 pad 1: ROW3 -> COL5
- D60 pad 1: ROW3 -> COL5
- MX22 pad 1: COL6 -> COL5
- MX24 pad 1: COL8 -> COL5
- MX37 pad 1: COL6 -> COL5
- MX39 pad 1: COL8 -> COL5
- MX52 pad 1: COL6 -> COL5
- MX54 pad 1: COL8 -> COL5
- MX7 pad 1: COL6 -> COL5
- MX9 pad 1: COL8 -> COL5

Commit message: updated the controller package
Parts:
- U1: footprint Package_QFP:TQFP-44_10x10mm_P0.8mm -> Package_QFP:TQFP-32_7x7mm_P0.8mm
- moved F1 279.3 mm to (194.5, 156.4)
- moved C1 241.4 mm to (248.3, 154.0)
- moved C3 241.4 mm to (211.0, 168.0)
- moved C5 241.4 mm to (215.4, 159.2)
- moved C6 241.4 mm to (211.0, 159.2)
- moved C7 241.4 mm to (241.2, 146.1)
- moved R2 241.4 mm to (211.0, 165.1)
- moved R3 241.4 mm to (253.9, 166.7)
- moved R4 241.4 mm to (215.4, 165.1)
- moved SW1 241.4 mm to (171.9, 160.9)
- moved Y1 241.4 mm to (179.3, 160.0)
- moved C2 241.4 mm to (225.3, 143.7)
- moved C4 241.4 mm to (211.0, 162.1)
- moved R1 241.4 mm to (215.4, 162.1)
- moved U1 195.5 mm to (234.9, 114.3)
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
Commit message: latest changes
Parts:
- added MX16-1: TAB, MX_Alps_Hybrid:MXOnly-1.5U-NoLED, F.Cu at (77.8, 68.3)
- added MX30-1: BACKSPACE, MX_Alps_Hybrid:MXOnly-1.5U-NoLED, F.Cu at (335.0, 68.3)
- added MX31-1: LAYER_UP, MX_Alps_Hybrid:MXOnly-1.25U-NoLED, F.Cu at (75.4, 87.3)
- added MX37-1: HOME, MX_Alps_Hybrid:MXOnly-1.25U-NoLED, F.Cu at (194.5, 87.3)
- added MX39-1: PAGE UP, MX_Alps_Hybrid:MXOnly-1.25U-NoLED, F.Cu at (218.3, 87.3)
- added MX45-1: RETURN, MX_Alps_Hybrid:MXOnly-1.25U-NoLED, F.Cu at (337.3, 87.3)
- MX16: value TAB -> TAB_orth
- MX30: value BACKSPACE -> BACKSPACE_orth
- MX31: value LAYER_UP -> LAYER_UP_orth
- MX37: value HOME -> HOME_orth
- MX39: value PAGE UP -> PAGE UP_orth
- MX45: value RETURN -> RETURN_orth

Commit message: flipped each component to the correct side, placed everything
Parts:
- removed D23, D38, D66, D67, D69: D_Small, Diode_SMD:D_0805_2012Metric
- removed MX23: Y, MX_Alps_Hybrid:MXOnly-1U-NoLED
- removed MX38, MX66, MX67, MX69: MX-1U, MX_Alps_Hybrid:MXOnly-1U-NoLED
- C1, C2, C3, C4, C5, C6, C7, D1, D10, D11, D12, D13, D14, D15, D16, D17, D18, D19, D2, D20, D21, D22, D24, D25, D26, D27, D28, D29, D3, D30, D31, D32, D33, D34, D35, D36, D37, D39, D4, D40, D41, D42, D43, D44, D45, D46, D47, D48, D49, D5, D50, D51, D52, D53, D54, D55, D56, D57, D58, D59, D6, D60, D61, D62, D63, D64, D65, D68, D7, D70, D71, D72, D73, D74, D75, D8, D9, F1, J1, R1, R2, R3, R4, SW1, Y1: moved to B.Cu
- U1: footprint Package_QFP:TQFP-32_7x7mm_P0.8mm -> Package_QFP:TQFP-48_7x7mm_P0.5mm; moved to B.Cu
- moved R3 204.8 mm to (80.0, 58.5), turned to 270 degrees
- moved R2 167.1 mm to (82.3, 58.5), turned to 270 degrees
- moved F1 153.3 mm to (80.9, 53.3), turned to 180 degrees
- moved SW1 102.6 mm to (106.3, 82.0), turned to 270 degrees
- moved Y1 81.2 mm to (235.0, 100.9), turned to 270 degrees
- moved C4 64.7 mm to (252.3, 112.3), turned to 180 degrees
- moved R1 60.0 mm to (252.3, 114.8)
- moved C6 57.8 mm to (233.6, 105.9), turned to 270 degrees
- moved C1 53.8 mm to (238.8, 101.0), turned to 90 degrees
- moved C3 52.6 mm to (235.1, 121.3), turned to 180 degrees
- moved C2 43.1 mm to (231.1, 101.0), turned to 270 degrees
- moved R4 41.1 mm to (240.2, 132.3), turned to 180 degrees
- moved C5 39.9 mm to (229.9, 122.0)
- moved C7 25.7 mm to (241.8, 120.4), turned to 90 degrees
- moved D55 7.10 mm to (253.0, 106.5), turned to 270 degrees
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
Commit message: started with traces.
Parts:
- C1, C2, C3, C4, C5, C6: footprint Capacitor_SMD:C_0805_2012Metric -> Capacitor_SMD:C_0201_0603Metric
- F1: footprint Fuse:Fuse_1206_3216Metric -> Fuse:Fuse_0805_2012Metric
- R2, R3: footprint Resistor_SMD:R_0805_2012Metric -> Resistor_SMD:R_0603_1608Metric
- moved D16 22.4 mm to (98.4, 72.9), turned to 90 degrees
- moved SW1 20.0 mm to (89.3, 92.5), turned to 180 degrees
- moved D65 19.1 mm to (172.2, 120.5)
- moved D32 13.8 mm to (89.7, 80.8)
- moved D30 13.7 mm to (337.5, 73.8), turned to 0 degrees
- moved D31 13.7 mm to (84.9, 81.0)
- moved D51 12.9 mm to (171.4, 111.3), turned to 90 degrees
- moved D14 12.9 mm to (323.9, 54.1), turned to 90 degrees
- moved D61 10.3 mm to (77.0, 131.0), turned to 180 degrees
- moved D46 10.3 mm to (76.8, 111.9), turned to 180 degrees
- moved D35 10.0 mm to (157.3, 91.9), turned to 90 degrees
- moved D36 10.0 mm to (176.4, 91.9), turned to 90 degrees
- moved D17 9.89 mm to (104.8, 72.9), turned to 90 degrees
- moved D18 9.89 mm to (123.8, 72.9), turned to 90 degrees
- moved D19 9.89 mm to (142.9, 72.9), turned to 90 degrees
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Connections:
- D46 pad 1: COL5 -> ROW3
- D47 pad 1: COL5 -> ROW3
- D48 pad 1: COL5 -> ROW3
- D49 pad 1: COL5 -> ROW3
- D50 pad 1: COL5 -> ROW3
- D51 pad 1: COL5 -> ROW3
- D52 pad 1: COL5 -> ROW3
- D53 pad 1: COL5 -> ROW3
- D54 pad 1: COL5 -> ROW3
- D55 pad 1: COL5 -> ROW3
- D56 pad 1: COL5 -> ROW3
- D57 pad 1: COL5 -> ROW3
- D58 pad 1: COL5 -> ROW3
- D59 pad 1: COL5 -> ROW3
- D60 pad 1: COL5 -> ROW3
- MX22 pad 1: COL5 -> COL6
- MX24 pad 1: COL5 -> COL8
- MX37 pad 1: COL5 -> COL6
- MX37-1 pad 1: COL5 -> COL6
- MX39 pad 1: COL5 -> COL8
- MX39-1 pad 1: COL5 -> COL8
- MX52 pad 1: COL5 -> COL6
- MX54 pad 1: COL5 -> COL8
- MX61 pad 1: Net-(MX61-Pad1) -> COL0
- MX62 pad 1: Net-(MX62-Pad1) -> COL1
- MX7 pad 1: COL5 -> COL6
- MX9 pad 1: COL5 -> COL8
Routing:
- net GND: track 0.00 -> 77.7 mm
- net Net-(D16-Pad2): track 0.00 -> 24.1 mm
- net Net-(D45-Pad2): track 0.00 -> 22.1 mm
- net Net-(D37-Pad2): track 0.00 -> 22.0 mm
- net Net-(D39-Pad2): track 0.00 -> 16.1 mm
- net Net-(D30-Pad2): track 0.00 -> 15.8 mm
- net Net-(D15-Pad2): track 0.00 -> 15.1 mm
- net VCC: track 0.00 -> 11.9 mm
- net Net-(D61-Pad2): track 0.00 -> 10.8 mm
- net Net-(D46-Pad2): track 0.00 -> 10.8 mm
- net Net-(D32-Pad2): track 0.00 -> 9.88 mm
- net Net-(D14-Pad2): track 0.00 -> 9.31 mm
- net Net-(D65-Pad2): track 0.00 -> 9.31 mm
- net Net-(D13-Pad2): track 0.00 -> 9.31 mm
- net Net-(D12-Pad2): track 0.00 -> 9.31 mm
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Other:
- net class Power added: clearance 0.2, trace_width 0.381, via_dia 0.8, via_drill 0.4

Commit message: further tracing
Parts:
- U1: footprint Package_QFP:TQFP-48_7x7mm_P0.5mm -> Package_QFP:TQFP-44_10x10mm_P0.8mm
- moved R4 25.3 mm to (216.3, 124.2), turned to 0 degrees
- moved C3 17.9 mm to (217.2, 122.3)
- moved D54 13.7 mm to (223.5, 99.6), turned to 270 degrees
- moved C5 12.8 mm to (217.2, 121.0), turned to 180 degrees
- moved C2 8.64 mm to (239.8, 101.0), turned to 90 degrees
- moved C1 8.26 mm to (230.5, 101.1), turned to 270 degrees
- moved R1 4.28 mm to (249.8, 111.3), turned to 270 degrees
- moved D55 2.09 mm to (250.6, 100.2), turned to 270 degrees
- moved C7 1.80 mm to (241.9, 120.9), turned to 180 degrees
- moved C6 1.39 mm to (234.6, 105.0), turned to 180 degrees
- moved U1 1.37 mm to (234.7, 114.9)
- moved C4 0.72 mm to (252.1, 111.6), turned to 270 degrees
- moved D51 0.19 mm to (171.4, 111.1)
Routing:
- net ROW3: track 0.00 -> 285.1 mm
- net ROW4: track 0.00 -> 278.4 mm
- net ROW0: track 0.00 -> 262.2 mm
- net ROW2: track 0.00 -> 246.4 mm
- net ROW1: track 0.00 -> 238.1 mm
- net COL4: track 0.00 -> 140.4 mm
- net COL3: track 0.00 -> 99.1 mm
- net COL2: track 0.00 -> 96.8 mm
- net COL0: track 0.00 -> 88.8 mm
- net COL1: track 0.00 -> 79.4 mm
- net COL5: track 0.00 -> 75.9 mm
- net COL6: track 0.00 -> 74.7 mm
- net GND: track 77.7 -> 128.9 mm
- net +5V: track 0.00 -> 36.3 mm
- net Net-(D70-Pad2): track 0.00 -> 19.1 mm
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
Commit message: further tracing applied
Connections:
- U1 pad 1: Net-(U1-Pad1) -> COL6
- U1 pad 10: Net-(U1-Pad10) -> ROW2
- U1 pad 11: Net-(U1-Pad11) -> COL9
- U1 pad 12: Net-(U1-Pad12) -> COL14
- U1 pad 18: Net-(U1-Pad18) -> COL5
- U1 pad 19: Net-(U1-Pad19) -> COL13
- U1 pad 20: Net-(U1-Pad20) -> COL12
- U1 pad 21: Net-(U1-Pad21) -> COL11
- U1 pad 22: Net-(U1-Pad22) -> COL10
- U1 pad 25: Net-(U1-Pad25) -> ROW4
- U1 pad 26: Net-(U1-Pad26) -> ROW3
- U1 pad 27: Net-(U1-Pad27) -> COL7
- U1 pad 28: Net-(U1-Pad28) -> COL8
- U1 pad 29: Net-(U1-Pad29) -> COL0
- U1 pad 30: Net-(U1-Pad30) -> COL1
- U1 pad 31: Net-(U1-Pad31) -> COL3
- U1 pad 32: Net-(U1-Pad32) -> COL4
- U1 pad 41: Net-(U1-Pad41) -> COL2
- U1 pad 8: Net-(U1-Pad8) -> ROW0
- U1 pad 9: Net-(U1-Pad9) -> ROW1
Routing:
- net COL14: track 0.00 -> 225.4 mm, vias 0 -> 1
- net COL13: track 0.00 -> 165.8 mm, vias 0 -> 1
- net COL12: track 0.00 -> 144.7 mm, vias 0 -> 1
- net COL11: track 0.00 -> 128.8 mm
- net COL10: track 0.00 -> 106.1 mm
- net COL9: track 0.00 -> 97.4 mm
- net COL8: track 0.00 -> 77.5 mm
- net ROW2: track 246.4 -> 267.1 mm, vias 0 -> 2
- net Net-(D30-Pad2): track 15.8 -> 35.0 mm, vias 0 -> 2
- net ROW4: track 278.4 -> 293.1 mm
